File: pcb/keypad.kicad_pcb (KiCad board)
At the start: 4 copper layers, 53 x 53 mm, 36 parts, among them SW1 KS33_SW_solder, SW2 KS33_SW_solder, SW3 KS33_SW_solder, SW4 KS33_SW_solder, SW5 KS33_SW_solder, SW6 KS33_SW_solder, SW7 KS33_SW_solder, SW8 KS33_SW_solder, SW9 KS33_SW_solder, U1 74AHCT1G125, U2 XIAO-ESP32-C6-DIP

Commit message: Set board stackup to 2 copper layers
The board was configured as a 4-layer stackup, but In1.Cu and In2.Cu
contained only through-hole pad and via annular rings — no routing or
zones.
Other:
- copper layers 4 -> 2
Changed lines of the file:
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@@
 	(layers
 		(0 "F.Cu" signal)
-		(4 "In1.Cu" signal)
-		(6 "In2.Cu" signal)
 		(2 "B.Cu" signal)
 		(9 "F.Adhes" user "F.Adhesive")
@@
 			)
 			(layer "dielectric 1"
-				(type "prepreg")
-				(thickness 0.1)
+				(type "core")
+				(thickness 1.51)
 				(material "FR4")
 				(epsilon_r 4.5)
-				(loss_tangent 0.02)
-			)
-			(layer "In1.Cu"
-				(type "copper")
-				(thickness 0.035)
-			)
-			(layer "dielectric 2"
-				(type "core")
-				(thickness 1.24)
-				(material "FR4")
-				(epsilon_r 4.5)
-				(loss_tangent 0.02)
-			)
-			(layer "In2.Cu"
-				(type "copper")
-				(thickness 0.035)
-			)
-			(layer "dielectric 3"
-				(type "prepreg")
-				(thickness 0.1)
-				(material "FR4")
-				(epsilon_r 4.5)
